File: pcbs/curtain_call/curtain_call.kicad_sch (KiCad schematic)
At the start: 1 part, among them U1 ESP32-H2

Commit message: pick component parts
Parts:
- added D1, D2: LED, LED_SMD:LED_0603_1608Metric, symbol Device:LED
- added M1: Motor_DC, symbol Motor:Motor_DC
- added R1, R2: R_Photo, OptoDevice:R_LDR_4.9x4.2mm_P2.54mm_Vertical, symbol Device:R_Photo
- added U2: DRV8833RTY, Package_DFN_QFN:Texas_RTY_WQFN-16-1EP_4x4mm_P0.65mm_EP2.1x2.1mm_ThermalVias, symbol Driver_Motor:DRV8833RTY
Connections:
- new net: U2.11 (GND), U2.17 (GND)

Commit message: feat: circuit diagram
Parts:
- removed U1: ESP32-H2, PCM_Espressif:QFN-32-1EP_4x4mm_P0.4mm_EP2.9x2.9mm, symbol PCM_Espressif:ESP32-H2
- removed U2: DRV8833RTY, Package_DFN_QFN:Texas_RTY_WQFN-16-1EP_4x4mm_P0.65mm_EP2.1x2.1mm_ThermalVias, symbol Driver_Motor:DRV8833RTY
- added C1: 10 µF, Capacitor_SMD:C_0402_1005Metric, symbol Device:C
- added C2: 0.1 µF, Capacitor_SMD:C_0805_2012Metric, symbol Device:C
- added J1: Conn_01x08, Connector_PinHeader_2.54mm:PinHeader_1x08_P2.54mm_Vertical, symbol Connector_Generic:Conn_01x08
- added R3: 15 kR, Resistor_SMD:R_0201_0603Metric, symbol Device:R
- added R4: 10 kR, Resistor_SMD:R_0201_0603Metric, symbol Device:R
- added R5, R6, R7, R8: R, symbol Device:R
- added U1: DRV8411ARTER, DRV8411ARTER:WQFN16_RTE_TEX, symbol DRV8411ARTER:DRV8411ARTER
- added U2: TLV9032DR, TLV9032DR:D0008A-IPC_A, symbol TLV9032DR:TLV9032DR
- M1: footprint (none) -> Connector_JST:JST_XH_B2B-XH-A_1x02_P2.50mm_Vertical
Connections:
- net GND: now reaches D1.1 (K)
- net GND: now also D2.1 (K), C1.1, C2.1, J1.2 (Pin_2), R3.2, R5.2, R6.2, U1.1 (PGNDA), U1.11 (GND), U1.17 (EPAD), U1.4 (PGNDB), U1.7 (BIN1), U1.8 (BIN2), U1.9 (BIPROPI), U2.4 (GND)
- net at D1.2 (A): now also R7.2
- net at M1.1 (+): now also U1.16 (AOUT1)
- net at M1.2 (-): now also U1.2 (AOUT2)
- net at D2.2 (A): now also R8.2
- net V_{EXT}: now reaches R2.1
- net V_{EXT}: now also R1.1, J1.3 (Pin_3), R4.1, U1.15 (VREF), U2.8 (VCC)
- net at R2.2: now also R5.1, U2.5 (IN2+)
- net at R1.2: now also R6.1, U2.3 (IN1+)
- new net IN_{1}: U1.14 (AIN1)
- new net IN_{2}: U1.13 (AIN2)
- new net LED_{1}: J1.4 (Pin_4), R7.1
- new net LED_{2}: J1.5 (Pin_5), R8.1
- new net LED_{OUT1}: J1.6 (Pin_6), U2.1 (OUT1)
- new net LED_{OUT2}: J1.7 (Pin_7), U2.7 (OUT2)
- new net VCC: C1.2, C2.2, J1.1 (Pin_1), U1.10 (VM)
- new net V_{Limit}: U2.2 (IN1-), U2.6 (IN2-)
- new net V_{PROPI}: J1.8 (Pin_8), R3.1, U1.12 (AIPROPI)
- new net nFAULT: R4.2, U1.6 (NFAULT)
Other:
- moved on the sheet: D1, D2, M1, R1, R2
